File: Design Files/SVG_ESC/ESC_01/MCU.kicad_sch (KiCad schematic)
At the start: 0 parts

Commit message: 0.01
Parts:
- added C1, C12, C13, C14, C2, C3, C4, C5, C6, C7: C, symbol Device:C
- added C10, C9: 2u2, symbol Device:C
- added C11, C16, C8: 100nF, symbol Device:C
- added C15, C17: 100n, symbol Device:C
- added D1: LED, symbol Device:LED
- added D2: LED_G, symbol Device:LED
- added D3: LED_R, symbol Device:LED
- added FB1: FerriteBead, symbol Device:FerriteBead
- added J1: Conn_01x06_Socket, symbol Connector:Conn_01x06_Socket
- added J2: Conn_01x03_Socket, symbol Connector:Conn_01x03_Socket
- added J3: Conn_01x08_Pin, symbol Connector:Conn_01x08_Pin
- added R1: 0R, symbol Device:R
- added R10, R7, R8: 2k2, symbol Device:R
- added R2, R3, R5, R6: R, symbol Device:R
- added R4: 1K, symbol Device:R
- added R9: 39k, symbol Device:R
- added SW1: SW_DIP_x01, symbol Switch:SW_DIP_x01
- added TH1: 10k, symbol Device:Thermistor_NTC
- added U1: STM32F405RGTx, Package_QFP:LQFP-64_10x10mm_P0.5mm, symbol MCU_ST_STM32F4:STM32F405RGTx
- added Y1: Crystal, symbol Device:Crystal
Connections:
- new net: R3.1, U1.6 (PH1)
- new net: C14.1, R3.2, Y1.1
- new net: C9.1, U1.31 (VCAP_1)
- new net: R6.1, U1.25 (PC5)
- new net: D3.2 (A), R6.2
- new net: J2.3 (Pin_3), R7.2
- new net: C17.1, R10.1, R9.2
- new net: C13.1, R2.2, Y1.2
- new net: R8.1, TH1.2
- new net: R1.2, U1.60 (BOOT0)
- new net: R2.1, U1.5 (PH0)
- new net: C10.1, U1.47 (VCAP_2)
- new net: D1.2 (A), R4.2
- new net: C15.1, R7.1
- new net: R5.1, U1.24 (PC4)
- new net: D2.2 (A), R5.2
- new net +3V3: C1.1, C11.1, C12.1, C16.1, C2.1, C3.1, C4.1, C5.1, C6.1, C7.1, FB1.1, FB1.2, J1.1 (Pin_1), J3.2 (Pin_2), R1.1, R4.1, TH1.1, U1.1 (VBAT), U1.13 (VDDA), U1.19 (VDD), U1.32 (VDD), U1.48 (VDD), U1.64 (VDD)
- new net +5V: J2.1 (Pin_1), J3.1 (Pin_1)
- new net +VDC: R9.1
- new net GND: C1.2, C10.2, C11.2, C12.2, C13.2, C14.2, C15.2, C16.2, C17.2, C2.2, C3.2, C4.2, C5.2, C6.2, C7.2, C8.2, C9.2, D1.1 (K), D2.1 (K), D3.1 (K), J1.3 (Pin_3), J2.2 (Pin_2), J3.3 (Pin_3), J3.8 (Pin_8), R10.2, R8.2, SW1.1, U1.12 (VSSA), U1.18 (VSS), U1.63 (VSS)
- new net NRST: C8.1, SW1.2, U1.7 (NRST)
- no-connect marks 0 -> 13
Other:
- note added: "100nF Decoupling Capacitors"
- note added: "10uF"
- note added: "ADC_TEMP"
- note added: "AN_IN"
- note added: "BR_S01"
- note added: "BR_S02"
- note added: "CAN_RX"
- note added: "CAN_TX"
- note added: "COMMUNICATION PROTOCALL"
- note added: "DC_CAL"
- note added: "EN_GATE"
- note added: "FAULT"
- note added: "H1"
- note added: "H2"
- note added: "H3"
- note added: "HALL_1"
- note added: "HALL_2"
- note added: "HALL_3"
- note added: "L1"
- note added: "L2"
- note added: "L3"
- note added: "LED_GREEN"
- note added: "LED_RED"
- note added: "MCU"
- note added: "MISO_ADC_EXT2"
- note added: "NRST"
- note added: "NRST Internally Pulled Up"
- note added: "NTC THERMISTOR"
- note added: "Programming/Debug"
- note added: "RX_SCI_MOSI"
- note added: "RX_SCL_MOSI"
- note added: "SCK_ADC_EXT"
- note added: "SENS1"
- note added: "SENS2"
- note added: "SENS3"
- note added: "SERVO"
- note added: "SUBSTITUTE WITH 100R IF USED AS SERVO OUTPUT"
- note added: "SWCLK"
- note added: "SWDIO"
- note added: "See BOOT Modes Table7"
- note added: "TEMP_MOTOR"
- note added: "TX_SDA_NSS"
- note added: "USB_DM"
- note added: "USB_DP"
- note added: "VOLTAGE DIVIDER"
- note added: "WHEN: VDC = 60V AN_IN = 3V204"
