File: Design Files/SVG_ESC/ESC_01/MOSFET_driver.kicad_sch (KiCad schematic)
At the start: 0 parts

Commit message: 0.1
Parts:
- added C18: 6800pF, symbol Device:C
- added C19: 120pF, symbol Device:C
- added C20, C21, C22, C23, C24, C25: 2u2, symbol Device:C
- added C26, C27, C28, C29, C30, C31, C32, C33, C36, C37, C38: 10u, symbol Device:C
- added C34: 1u, symbol Device:C
- added C35, C39, C40, C41: 100n, symbol Device:C
- added D4: BAT60A, Diode_SMD:D_SOD-323, symbol Diode:BAT60A
- added D5: PMEG6020, Diode_SMD:Nexperia_CFP3_SOD-123W, symbol Diode:PMEG6020ER
- added L1: 22u, symbol Device:L
- added R11: 205k, symbol Device:R
- added R12: 16k2, symbol Device:R
- added R13, R16, R19, R21, R23: 18k, symbol Device:R
- added R14, R17: 3k3, symbol Device:R
- added R15: 10k, symbol Device:R
- added R18: 1M, symbol Device:R
- added R20, R22, R24: 2K2, symbol Device:R
- added U2: DRV8302DCA, DCA56_6P35X3P61, symbol DRV8302:DRV8302DCA
Connections:
- new net: C36.1, C37.1, C38.1, D4.2 (A), L1.2, R16.1
- new net: R23.2, R24.1
- new net: R13.2, R14.1, U2.3 (VSENSE)
- new net: C35.2, D5.1 (K), L1.1, U2.50 (PH), U2.51 (PH)
- new net: R18.1, U2.49 (BIAS)
- new net: R11.1, U2.1 (RT_CLK)
- new net: C20.1, C21.1, U2.11 (OC_ADJ)
- new net: C24.1, U2.14 (CP1)
- new net: C24.2, U2.15 (CP2)
- new net: C19.1, R12.1, U2.2 (COMP)
- new net: C25.1, U2.27 (AVDD)
- new net: R16.2, R17.1
- new net: R21.2, R22.1
- new net: C35.1, U2.52 (BST_BK)
- new net: R19.2, R20.1
- new net: C18.1, R12.2
- new net: R15.2, U2.7 (DTC)
- new net: C22.1, C23.1, U2.13 (GVDD)
- new net +5V: D4.1 (K), R13.1
- new net +VDC: C26.1, C27.1, C28.1, C29.1, C30.1, C31.1, C32.1, C33.1, C34.1, U2.29 (PVDD1), U2.53 (PVDD2), U2.54 (PVDD2)
- new net DC_CAL: U2.12 (DC_CAL)
- new net Fault: U2.6 (*FAULT)
- new net GND: C18.2, C19.2, C20.2, C21.2, C22.2, C23.2, C25.2, C26.2, C27.2, C28.2, C29.2, C30.2, C31.2, C32.2, C33.2, C34.2, C36.2, C37.2, C38.2, D5.2 (A), R11.2, R14.2, R15.1, R17.2, R18.2, R20.2, R22.2, R24.2, U2.10 (GAIN), U2.28 (AGND), U2.57 (EPAD), U2.8 (M_PWM)
- new net H3_VS: R19.1, R21.1, R23.1
- no-connect marks 0 -> 4
Other:
- note added: "+3V3"
- note added: "+5V_DRV"
- note added: "1u DECOUPLER PLACE AS CLOSE AS POSSIBLE TO IC"
- note added: "BIAS"
- note added: "BOOTSTRAP CAPs"
- note added: "BR_S01"
- note added: "BR_S02"
- note added: "BST_A"
- note added: "BST_B"
- note added: "BST_BK"
- note added: "BST_C"
- note added: "BULK CAPACITANCE KEEP AS CLOSE AS POSSIBLE TO THE IC AND TO THE DRIVER INPUT LOOP"
- note added: "DE_CAL"
- note added: "DVDD"
- note added: "EN_GATE"
- note added: "FAULT"
- note added: "H1"
- note added: "H1_LOW"
- note added: "H1_VS"
- note added: "H2"
- note added: "H2_LOW"
- note added: "H2_VS"
- note added: "H3"
- note added: "H3_LOW"
- note added: "H3_VS"
- note added: "Hx_VS"
- note added: "INPUT PORTS"
- note added: "KEEP AWAY FROM NOISY TRACKS AND COMPONENTS"
- note added: "L1"
- note added: "L2"
- note added: "L3"
- note added: "MCU SENSING FEEDBACK FOR EACH PHASE"
- note added: "MOSFET Driver"
- note added: "M_H1"
- note added: "M_H2"
- note added: "M_H3"
- note added: "M_L1"
- note added: "M_L2"
- note added: "M_L3"
- note added: "OUTPUT PORTS"
- note added: "PH"
- note added: "PHASE_1"
- note added: "PHASE_2"
- note added: "PHASE_3"
- note added: "S1_N"
- note added: "S1_P"
- note added: "S2_N"
- note added: "S2_P"
- note added: "SENSE 1 - PHASE 1"
- note added: "SENSE 2 - PHASE 2"
- note added: "VSENSE"

Commit message: 0.1
Changed lines of the file:
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@@
 	(global_label "SENS1"
 		(shape input)
-		(at 223.52 135.89 0)
+		(at 222.25 135.89 0)
 		(fields_autoplaced yes)
 		(effects
@@
 		)
 		(property "Intersheetrefs" "${INTERSHEET_REFS}"
-			(at 232.6132 135.89 0)
+			(at 231.3432 135.89 0)
 			(effects
 				(font
