File: Design Files/SVG_ESC/ESC_01/MOSFETs.kicad_sch (KiCad schematic)
At the start: 0 parts

Commit message: 0.1
Parts:
- added C42, C43: 2n2, symbol Device:C
- added J4, J5, J6: Conn_01x01, symbol Connector:Conn_01x01_Socket
- added NT1, NT2, NT3, NT4, NT5, NT6, NT7, NT8: NetTie_2, symbol Device:NetTie_2
- added Q1, Q2, Q3, Q4, Q5, Q6: HSBA15810C, Package_TO_SOT_SMD:LFPAK33, symbol Transistor_FET:BUK7M6R3-40EX
- added R25, R26, R31, R32, R37, R38: 4R7, symbol Device:R
- added R27, R35, R41: 39k, symbol Device:R
- added R28, R36: 0R001, symbol Device:R
- added R29, R30, R33, R34: 100R, symbol Device:R
Connections:
- new net: NT4.2, Q3.1 (S), Q3.2 (S), Q3.3 (S), Q4.5 (D)
- new net: NT6.2, R34.1, R36.1
- new net: Q4.4 (G), R32.2, R35.2
- new net: Q6.4 (G), R38.2, R41.2
- new net: NT3.2, R28.1, R30.1
- new net: NT5.1, R33.1, R36.2
- new net: NT5.2, Q4.1 (S), Q4.2 (S), Q4.3 (S)
- new net: NT7.2, Q5.1 (S), Q5.2 (S), Q5.3 (S), Q6.5 (D)
- new net: NT8.2, Q6.1 (S), Q6.2 (S), Q6.3 (S)
- new net: Q3.4 (G), R31.2
- new net: Q1.4 (G), R25.2
- new net: Q2.4 (G), R26.2, R27.2
- new net: NT2.1, R28.2, R29.1
- new net: NT2.2, Q2.1 (S), Q2.2 (S), Q2.3 (S)
- new net: C43.1, R33.2
- new net: C43.2, R34.2
- new net: NT1.2, Q1.1 (S), Q1.2 (S), Q1.3 (S), Q2.5 (D)
- new net: C42.1, R29.2
- new net: C42.2, R30.2
- new net: Q5.4 (G), R37.2
- new net +VDC: Q1.5 (D), Q3.5 (D), Q5.5 (D)
- new net GND: NT3.1, NT6.1, NT8.1, R27.1, R35.1, R41.1
Other:
- note added: "H1_LOW"
- note added: "H1_VS"
- note added: "H2_LOW"
- note added: "H2_VS"
- note added: "H3_LOW"
- note added: "H3_VS"
- note added: "Hx_VS"
- note added: "MCU SENSING FEEDBACK FOR EACH PHASE"
- note added: "MH_1"
- note added: "MH_1_RG"
- note added: "MH_2"
- note added: "MH_2_RG"
- note added: "MH_3"
- note added: "MH_3_RG"
- note added: "ML_1"
- note added: "ML_1_RG"
- note added: "ML_2"
- note added: "ML_2_RG"
- note added: "ML_3"
- note added: "ML_3_RG"
- note added: "MOSFETs"
- note added: "M_H1"
- note added: "M_H2"
- note added: "M_H3"
- note added: "M_L1"
- note added: "M_L2"
- note added: "M_L3"
- note added: "OUTPUT PHASE 1"
- note added: "OUTPUT PHASE 2"
- note added: "OUTPUT PHASE 3"
- note added: "PHASE 1"
- note added: "PHASE 2"
- note added: "PHASE 3"
- note added: "PHASE_1"
- note added: "PHASE_2"
- note added: "PHASE_3"
- note added: "PLACE AS CLOSE AS POSSIBLE TO THE BULK CAPACITANCE"
- note added: "Q_CONTROL"
- note added: "Q_SOURCES"
- note added: "ROUTE AS KELVING CONNECTIONS"
- note added: "S1_N"
- note added: "S1_P"
- note added: "S2_N"
- note added: "S2_P"
- note added: "SENSE 1"
- note added: "SENSE 2"
- note added: "SH1_N"
- note added: "SH1_P"
- note added: "SH2_N"
- note added: "SH2_P"
