File: Projects/ESP32_01/ESP32_01.kicad_sch (KiCad schematic)
At the start: 17 parts, among them J1 USB_B_Micro, SW1 SW_Push, SW2 SW_Push, U1 ESP32-S3-MINI-1, U2 D3V3XA4B10LP, U3 TLV75801PDRV

Commit message: P2
Parts:
- BOOT1: renamed from SW2; value SW_Push -> ~; footprint (none) -> Button_Switch_THT:SW_PUSH_6mm
- C1, C2, C3, C4, C5, C6: footprint (none) -> Capacitor_SMD:C_0805_2012Metric
- D1, R2: footprint (none) -> LED_SMD:LED_0805_2012Metric
- J1: footprint (none) -> Connector_USB:USB_Micro-B_Amphenol_10118193-0002LF_Horizontal
- R1, R3, R4: footprint (none) -> Resistor_SMD:R_0805_2012Metric
- RESET1: renamed from SW1; value SW_Push -> ~; footprint (none) -> Button_Switch_THT:SW_PUSH_6mm
Other:
- note added: "GPIO0"
- moved on the sheet: RESET1
Changed lines of the file:
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@@
+	)
+	(junction
+		(at 154.94 55.88)
+		(diameter 0)
+		(color 0 0 0 0)
 	)
 	(junction
@@
 	(wire
 		(pts
+			(xy 154.94 55.88) (xy 154.94 54.61)
+		)
+		(stroke
+			(width 0)
+			(type default)
+		)
+	)
+	(wire
+		(pts
 			(xy 123.19 171.45) (xy 139.7 171.45)
 		)
@@
 	(wire
 		(pts
-			(xy 154.94 54.61) (xy 154.94 58.42)
-		)
-		(stroke
-			(width 0)
-			(type default)
-		)
-	)
-	(wire
-		(pts
 			(xy 154.94 41.91) (xy 154.94 34.29)
 		)
@@
 	(wire
 		(pts
+			(xy 154.94 55.88) (xy 154.94 58.42)
+		)
+		(stroke
+			(width 0)
+			(type default)
+		)
+	)
+	(wire
+		(pts
 			(xy 59.69 76.2) (xy 59.69 81.28)
 		)
@@
 	(wire
 		(pts
-			(xy 139.7 54.61) (xy 139.7 69.85)
+			(xy 139.7 55.88) (xy 139.7 69.85)
 		)
 		(stroke
@@
 	(wire
 		(pts
-			(xy 149.86 54.61) (xy 154.94 54.61)
+			(xy 149.86 55.88) (xy 154.94 55.88)
 		)
 		(stroke
@@
 		(exclude_from_sim no)
 		(at 76.454 67.818 0)
+		(effects
+			(font
+				(size 1.27 1.27)
+			)
+		)
+	)
+	(text "GPIO0"
+		(exclude_from_sim no)
+		(at 166.624 70.104 0)
 		(effects
 			(font
@@
 			)
 		)
-		(property "Footprint" ""
+		(property "Footprint" "Resistor_SMD:R_0805_2012Metric"
 			(at 121.412 163.83 90)
 			(effects
@@
 	(symbol
 		(lib_id "Switch:SW_Push")
-		(at 144.78 54.61 0)
+		(at 144.78 55.88 0)
 		(unit 1)
 		(exclude_from_sim no)
@@
 		(on_board yes)
 		(dnp no)
-		(fields_autoplaced yes)
-		(property "Reference" "SW1"
-			(at 144.78 46.99 0)
-			(effects
-				(font
-					(size 1.27 1.27)
-				)
-			)
-		)
-		(property "Value" "SW_Push"
-			(at 144.78 49.53 0)
-			(effects
-				(font
-					(size 1.27 1.27)
-				)
-			)
-		)
-		(property "Footprint" ""
-			(at 144.78 49.53 0)
+		(property "Reference" "RESET1"
+			(at 145.034 51.308 0)
+			(effects
+				(font
+					(size 1.27 1.27)
+				)
+			)
+		)
+		(property "Value" "~"
+			(at 144.78 50.8 0)
+			(effects
+				(font
+					(size 1.27 1.27)
+				)
+			)
+		)
+		(property "Footprint" "Button_Switch_THT:SW_PUSH_6mm"
+			(at 144.78 50.8 0)
 			(effects
 				(font
@@
 		)
 		(property "Datasheet" "~"
-			(at 144.78 49.53 0)
+			(at 144.78 50.8 0)
 			(effects
 				(font
@@
 		)
 		(property "Description" "Push button switch, generic, two pins"
-			(at 144.78 54.61 0)
+			(at 144.78 55.88 0)
 			(effects
 				(font
@@
 			(project ""
 				(path "/e7686582-131b-41c3-aca7-fbe57ebb66ed"
-					(reference "SW1")
+					(reference "RESET1")
 					(unit 1)
 				)
@@
 		(on_board yes)
 		(dnp no)
-		(fields_autoplaced yes)
-		(property "Reference" "SW2"
-			(at 146.05 76.2 0)
-			(effects
-				(font
-					(size 1.27 1.27)
-				)
-			)
-		)
-		(property "Value" "SW_Push"
+		(property "Reference" "BOOT1"
+			(at 146.05 79.502 0)
+			(effects
+				(font
+					(size 1.27 1.27)
+				)
+			)
+		)
+		(property "Value" "~"
 			(at 146.05 78.74 0)
 			(effects
@@
 			)
 		)
-		(property "Footprint" ""
+		(property "Footprint" "Button_Switch_THT:SW_PUSH_6mm"
 			(at 146.05 78.74 0)
 			(effects
@@
 			(project "ESP32_01"
 				(path "/e7686582-131b-41c3-aca7-fbe57ebb66ed"
-					(reference "SW2")
+					(reference "BOOT1")
 					(unit 1)
 				)
@@
 			)
 		)
-		(property "Footprint" ""
+		(property "Footprint" "Capacitor_SMD:C_0805_2012Metric"
 			(at 157.1752 92.71 0)
 			(effects
@@
 			)
 		)
-		(property "Footprint" ""
+		(property "Footprint" "Capacitor_SMD:C_0805_2012Metric"
 			(at 72.0852 154.94 0)
 			(effects
@@
 			)
 		)
-		(property "Footprint" ""
+		(property "Footprint" "Capacitor_SMD:C_0805_2012Metric"
 			(at 216.8652 58.42 0)
 			(effects
@@
 			)
 		)
-		(property "Footprint" ""
+		(property "Footprint" "Connector_USB:USB_Micro-B_Amphenol_10118193-0002LF_Horizontal"
 			(at 63.5 67.31 0)
 			(effects
@@
 			)
 		)
-		(property "Footprint" ""
+		(property "Footprint" "LED_SMD:LED_0805_2012Metric"
 			(at 160.02 157.48 0)
 			(effects
@@
 			)
 		)
-		(property "Footprint" ""
+		(property "Footprint" "Capacitor_SMD:C_0805_2012Metric"
 			(at 155.9052 66.04 0)
 			(effects
@@
 			)
 		)
-		(property "Footprint" ""
+		(property "Footprint" "Capacitor_SMD:C_0805_2012Metric"
 			(at 140.6652 158.75 0)
 			(effects
@@
 			)
 		)
-		(property "Footprint" ""
+		(property "Footprint" "Capacitor_SMD:C_0805_2012Metric"
 			(at 234.6452 58.42 0)
 			(effects
@@
 			)
 		)
-		(property "Footprint" ""
+		(property "Footprint" "Resistor_SMD:R_0805_2012Metric"
 			(at 151.13 145.288 90)
 			(effects
@@
 			)
 		)
-		(property "Footprint" ""
+		(property "Footprint" "LED_SMD:LED_0805_2012Metric"
 			(at 121.412 149.86 90)
 			(effects
@@
 			)
 		)
-		(property "Footprint" ""
+		(property "Footprint" "Resistor_SMD:R_0805_2012Metric"
 			(at 153.162 45.72 90)
 			(effects
